Commit message: gz simulation with ros2 control implemented

File: src/skywarden_description/urdf/body.xacro (robot description, xacro)
@@ -5,13 +5,17 @@
     <xacro:property name="base_ly" value="0.3" />
     <xacro:property name="base_lz" value="0.05" />
+    <xacro:property name="base_mass" value="0.8" />
     <xacro:property name="yaw_lx" value="0.2" />
     <xacro:property name="yaw_ly" value="0.2" />
     <xacro:property name="yaw_lz" value="0.05" />
+    <xacro:property name="yaw_mass" value="0.2" />
     <xacro:property name="stand_lx" value="0.05" />
     <xacro:property name="stand_ly" value="0.02" />
     <xacro:property name="stand_lz" value="0.15" />
+    <xacro:property name="stand_mass" value="0.1" />
     <xacro:property name="pitch_lx" value="0.05" />
     <xacro:property name="pitch_ly" value="0.1" />
     <xacro:property name="pitch_lz" value="0.02" />
+    <xacro:property name="pitch_mass" value="0.1" />
     <!-- END_SPECS -->
     <link name="footprint" />
@@ -24,4 +28,12 @@
             <material name="red" />
         </visual>
+        <collision>
+            <origin xyz="0 0 0" rpy="0 0 0" />
+            <geometry>
+                <box size="${base_lx} ${base_ly} ${base_lz}" />
+            </geometry>
+        </collision>
+        <xacro:box_inertial m="${base_mass}" lx="${base_lx}" ly="${base_ly}" lz="${base_lz}"
+            o_xyz="0 0 0" o_rpy="0 0 0" />
     </link>
     <joint name="base_footprint_joint" type="fixed">
@@ -38,4 +50,12 @@
             <material name="green" />
         </visual>
+        <collision>
+            <origin xyz="0 0 ${yaw_lz / 2}" rpy="0 0 0" />
+            <geometry>
+                <box size="${yaw_lx} ${yaw_ly} ${yaw_lz}" />
+            </geometry>
+        </collision>
+        <xacro:box_inertial m="${yaw_mass}" lx="${yaw_lx}" ly="${yaw_ly}" lz="${yaw_lz}"
+            o_xyz="0 0 ${yaw_lz / 2}" o_rpy="0 0 0" />
     </link>
     <joint name="yaw_base_joint" type="revolute">
@@ -56,4 +76,12 @@
             <material name="black" />
         </visual>
+        <collision>
+            <origin xyz="0 0 ${stand_lz / 2}" rpy="0 0 0" />
+            <geometry>
+                <box size="${stand_lx} ${stand_ly} ${stand_lz}" />
+            </geometry>
+        </collision>
+        <xacro:box_inertial m="${stand_mass}" lx="${stand_lx}" ly="${stand_ly}" lz="${stand_lz}"
+            o_xyz="0 0 ${stand_lz / 2}" o_rpy="0 0 0" />
     </link>
     <joint name="lstand_yaw_joint" type="fixed">
@@ -70,4 +98,12 @@
             <material name="black" />
         </visual>
+        <collision>
+            <origin xyz="0 0 ${stand_lz / 2}" rpy="0 0 0" />
+            <geometry>
+                <box size="${stand_lx} ${stand_ly} ${stand_lz}" />
+            </geometry>
+        </collision>
+        <xacro:box_inertial m="${stand_mass}" lx="${stand_lx}" ly="${stand_ly}" lz="${stand_lz}"
+            o_xyz="0 0 ${stand_lz / 2}" o_rpy="0 0 0" />
     </link>
     <joint name="rstand_yaw_joint" type="fixed">
@@ -84,4 +120,12 @@
             <material name="blue" />
         </visual>
+        <collision>
+            <origin xyz="0 0 0" rpy="0 0 0" />
+            <geometry>
+                <box size="${pitch_lx} ${pitch_ly} ${pitch_lz}" />
+            </geometry>
+        </collision>
+        <xacro:box_inertial m="${pitch_mass}" lx="${pitch_lx}" ly="${pitch_ly}" lz="${pitch_lz}"
+            o_xyz="0 0 0" o_rpy="0 0 0" />
     </link>
     <joint name="pitch_base_joint" type="revolute">

File: src/skywarden_description/urdf/skywarden.urdf.xacro (robot description, xacro)
@@ -2,4 +2,7 @@
 <robot xmlns:xacro="http://www.ros.org/wiki/xacro" name="skywarden">
     <xacro:include filename="./materials.xacro" />
+    <xacro:include filename="./inertials.xacro" />
     <xacro:include filename="./body.xacro" />
+    <xacro:include filename="./gz_plugins.xacro" />
+    <xacro:include filename="./gz.ros2control.xacro" />
 </robot>

Commit message: added camera and shooter links

File: src/skywarden_description/urdf/body.xacro (robot description, xacro)
@@ -14,8 +14,15 @@
     <xacro:property name="stand_lz" value="0.15" />
     <xacro:property name="stand_mass" value="0.1" />
-    <xacro:property name="pitch_lx" value="0.05" />
-    <xacro:property name="pitch_ly" value="0.1" />
-    <xacro:property name="pitch_lz" value="0.02" />
+    <xacro:property name="pitch_lx" value="0.02" />
+    <xacro:property name="pitch_ly" value="0.15" />
+    <xacro:property name="pitch_lz" value="0.13" />
     <xacro:property name="pitch_mass" value="0.1" />
+    <xacro:property name="shooter_lx" value="0.07" />
+    <xacro:property name="shooter_ly" value="0.05" />
+    <xacro:property name="shooter_lz" value="0.05" />
+    <xacro:property name="shooter_mass" value="0.02" />
+    <xacro:property name="camera_lx" value="0.02" />
+    <xacro:property name="camera_ly" value="0.04" />
+    <xacro:property name="camera_lz" value="0.04" />
     <!-- END_SPECS -->
     <link name="footprint" />
@@ -114,5 +121,5 @@
     <link name="pitch_link">
         <visual>
-            <origin xyz="0 0 0" rpy="0 0 0" />
+            <origin xyz="0 0 0.02" rpy="0 0 0" />
             <geometry>
                 <box size="${pitch_lx} ${pitch_ly} ${pitch_lz}" />
@@ -137,3 +144,32 @@
         have holding toruqe of 0.3 N*m-->
     </joint>
+    <link name="shooter_link">
+        <visual>
+            <origin xyz="0 0 0" rpy="0 0 0" />
+            <geometry>
+                <box size="${shooter_lx} ${shooter_ly} ${shooter_lz}" />
+            </geometry>
+            <material name="white" />
+        </visual>
+    </link>
+    <joint name="shooter_pitch_joint" type="fixed">
+        <origin xyz="${(pitch_lx + shooter_lx) / 2} 0 0" rpy="0 0 0"/>
+        <parent link="pitch_link"/>
+        <child link="shooter_link"/>
+    </joint>
+    <!-- Camera -->
+    <link name="camera_link">
+        <visual>
+            <origin xyz="0.0 0 0" rpy="0 0 0"/>
+            <geometry>
+                <box size="${camera_lx} ${camera_ly} ${camera_lz}"/>
+            </geometry>
+            <material name="black" />
+        </visual>
+    </link>
+    <joint name="camera_pitch_link" type="fixed">
+        <origin xyz="${(pitch_lx + camera_lx) / 2} 0 ${pitch_lz - camera_lz * 1.7}" rpy="0 0 0" />
+        <parent link="pitch_link" />
+        <child link="camera_link" />
+    </joint>
 </robot>

File: src/skywarden_description/urdf/materials.xacro (robot description, xacro)
@@ -3,4 +3,7 @@
     <material name="black">
         <color rgba="0 0 0 1.0"/>
+    </material>
+    <material name="white">
+        <color rgba="1 1 1 1.0"/>
     </material>
     <material name="red">

Commit message: Added ballistic arc visualization and simulating drone in rviz

File: src/skywarden_description/urdf/body.xacro (robot description, xacro)
@@ -18,8 +18,8 @@
     <xacro:property name="pitch_lz" value="0.13" />
     <xacro:property name="pitch_mass" value="0.1" />
-    <xacro:property name="shooter_lx" value="0.07" />
-    <xacro:property name="shooter_ly" value="0.05" />
-    <xacro:property name="shooter_lz" value="0.05" />
-    <xacro:property name="shooter_mass" value="0.02" />
+    <xacro:property name="muzzle_lx" value="0.07" />
+    <xacro:property name="muzzle_ly" value="0.05" />
+    <xacro:property name="muzzle_lz" value="0.05" />
+    <xacro:property name="muzzle_mass" value="0.02" />
     <xacro:property name="camera_lx" value="0.02" />
     <xacro:property name="camera_ly" value="0.04" />
@@ -144,17 +144,17 @@
         have holding toruqe of 0.3 N*m-->
     </joint>
-    <link name="shooter_link">
+    <link name="muzzle_link">
         <visual>
             <origin xyz="0 0 0" rpy="0 0 0" />
             <geometry>
-                <box size="${shooter_lx} ${shooter_ly} ${shooter_lz}" />
+                <box size="${muzzle_lx} ${muzzle_ly} ${muzzle_lz}" />
             </geometry>
             <material name="white" />
         </visual>
     </link>
-    <joint name="shooter_pitch_joint" type="fixed">
-        <origin xyz="${(pitch_lx + shooter_lx) / 2} 0 0" rpy="0 0 0"/>
+    <joint name="muzzle_pitch_joint" type="fixed">
+        <origin xyz="${(pitch_lx + muzzle_lx) / 2} 0 0" rpy="0 0 0"/>
         <parent link="pitch_link"/>
-        <child link="shooter_link"/>
+        <child link="muzzle_link"/>
     </joint>
     <!-- Camera -->

Commit message: Added Predictive Lead equation and drone orbitting around

File: src/skywarden_description/urdf/body.xacro (robot description, xacro)
@@ -71,5 +71,5 @@
         <child link="yaw_link" />
         <axis xyz="0 0 1" />
-        <limit lower="${-pi/2}" upper="${pi/2}" effort="30" velocity="${pi}" /> <!-- Nema 17 motor
+        <limit lower="0" upper="${pi}" effort="30" velocity="${pi}" /> <!-- Nema 17 motor
         have holding toruqe of 0.3 N*m-->
     </joint>

Commit message: added pid controller (still bad)

File: src/skywarden_description/urdf/body.xacro (robot description, xacro)
@@ -66,10 +66,10 @@
             o_xyz="0 0 ${yaw_lz / 2}" o_rpy="0 0 0" />
     </link>
-    <joint name="yaw_base_joint" type="revolute">
+    <joint name="yaw_base_joint" type="continuous">
         <origin xyz="0 0 ${base_lz / 2}" rpy="0 0 0" />
         <parent link="base_link" />
         <child link="yaw_link" />
         <axis xyz="0 0 1" />
-        <limit lower="0" upper="${pi}" effort="30" velocity="${pi}" /> <!-- Nema 17 motor
+        <limit effort="30" velocity="${pi}" /> <!-- Nema 17 motor
         have holding toruqe of 0.3 N*m-->
     </joint>
